File: Lab 8/Experiment 1/schematic 1.sch (EAGLE design)
At the start: 22 parts, among them IC1 STM32F10XCXT6, J1 CORTEX_JTAG_DEBUG_PTH, Q1 8MHz

Commit message: Lab 8
Parts:
- removed R1: 390, adafruit:FLIPFLOP-RES
- removed R2: 10kOhm, adafruit:FLIPFLOP-RES
- added R3: 390, adafruit:R-US_MELF0102W
- added R4: 10KOhm, adafruit:R-US_MELF0102W
Connections:
- net N$3: now also R4.1; no longer R2.1
- net N$4: now also R3.2; no longer R1.2
- net N$5: now also R3.1; no longer R1.1
- net N$6: now also R4.2; no longer R2.2
Changed lines of the file:
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@@
 <part name="C8" library="capacitor-wima" library_urn="urn:adsk.eagle:library:116" deviceset="C" device="2,5-3" package3d_urn="urn:adsk.eagle:package:5436/1" value="20pF"/>
 <part name="C9" library="capacitor-wima" library_urn="urn:adsk.eagle:library:116" deviceset="C" device="2,5-3" package3d_urn="urn:adsk.eagle:package:5436/1" value="20pF"/>
-<part name="R1" library="adafruit" deviceset="FLIPFLOP-RES" device="" value="390"/>
-<part name="R2" library="adafruit" deviceset="FLIPFLOP-RES" device="" value="10kOhm"/>
 <part name="S1" library="adafruit" deviceset="EG1213" device=""/>
 <part name="SUPPLY4" library="SparkFun-PowerSymbols" deviceset="VDD" device=""/>
@@
 <part name="JP2" library="adafruit" deviceset="PINHD-1X8" device="-3.5MM"/>
 <part name="JP3" library="adafruit" deviceset="PINHD-1X8" device="-3.5MM"/>
+<part name="R3" library="adafruit" deviceset="R-US_" device="MELF0102W" value="390"/>
+<part name="R4" library="adafruit" deviceset="R-US_" device="MELF0102W" value="10KOhm"/>
 </parts>
 <sheets>
@@
 <attribute name="VALUE" x="159.639" y="54.864" size="1.778" layer="96" rot="R90"/>
 </instance>
-<instance part="R1" gate="G$1" x="137.16" y="53.34" smashed="yes">
-<attribute name="NAME" x="133.35" y="54.8386" size="1.778" layer="95"/>
-<attribute name="VALUE" x="133.35" y="50.038" size="1.778" layer="96"/>
-</instance>
-<instance part="R2" gate="G$1" x="129.54" y="142.24" smashed="yes">
-<attribute name="NAME" x="125.73" y="143.7386" size="1.778" layer="95"/>
-<attribute name="VALUE" x="125.73" y="138.938" size="1.778" layer="96"/>
-</instance>
 <instance part="S1" gate="1" x="139.7" y="137.16" smashed="yes" rot="R270">
 <attribute name="NAME" x="137.795" y="145.415" size="1.778" layer="95"/>
@@
 <attribute name="NAME" x="11.43" y="32.385" size="1.778" layer="95" rot="R180"/>
 <attribute name="VALUE" x="11.43" y="58.42" size="1.778" layer="96" rot="R180"/>
+</instance>
+<instance part="R3" gate="G$1" x="134.62" y="45.72" smashed="yes">
+<attribute name="NAME" x="130.81" y="47.2186" size="1.778" layer="95"/>
+<attribute name="VALUE" x="130.81" y="42.418" size="1.778" layer="96"/>
+</instance>
+<instance part="R4" gate="G$1" x="127" y="137.16" smashed="yes">
+<attribute name="NAME" x="123.19" y="138.6586" size="1.778" layer="95"/>
+<attribute name="VALUE" x="123.19" y="133.858" size="1.778" layer="96"/>
 </instance>
 </instances>
@@
 <net name="N$4" class="0">
 <segment>
-<pinref part="R1" gate="G$1" pin="2"/>
 <pinref part="C9" gate="G$1" pin="1"/>
-<wire x1="142.24" y1="53.34" x2="144.78" y2="53.34" width="0.1524" layer="91"/>
 <pinref part="Q1" gate="G$1" pin="1"/>
 <wire x1="144.78" y1="53.34" x2="152.4" y2="53.34" width="0.1524" layer="91"/>
 <wire x1="144.78" y1="55.88" x2="144.78" y2="53.34" width="0.1524" layer="91"/>
 <junction x="144.78" y="53.34"/>
-</segment>
-</net>
-<net name="N$5" class="0">
-<segment>
-<pinref part="IC1" gate="PORTD/OSC" pin="PD1/OSC=&gt;"/>
-<wire x1="121.92" y1="55.88" x2="127" y2="55.88" width="0.1524" layer="91"/>
-<wire x1="127" y1="55.88" x2="127" y2="53.34" width="0.1524" layer="91"/>
-<pinref part="R1" gate="G$1" pin="1"/>
-<wire x1="127" y1="53.34" x2="132.08" y2="53.34" width="0.1524" layer="91"/>
-</segment>
-</net>
-<net name="N$3" class="0">
-<segment>
-<pinref part="IC1" gate="RESET" pin="BOOT0"/>
-<pinref part="R2" gate="G$1" pin="1"/>
-<wire x1="121.92" y1="144.78" x2="121.92" y2="142.24" width="0.1524" layer="91"/>
-<wire x1="121.92" y1="142.24" x2="124.46" y2="142.24" width="0.1524" layer="91"/>
-</segment>
-</net>
-<net name="N$6" class="0">
-<segment>
-<pinref part="R2" gate="G$1" pin="2"/>
-<pinref part="S1" gate="1" pin="P"/>
-<wire x1="134.62" y1="142.24" x2="134.62" y2="137.16" width="0.1524" layer="91"/>
+<pinref part="R3" gate="G$1" pin="2"/>
+<wire x1="139.7" y1="45.72" x2="144.78" y2="45.72" width="0.1524" layer="91"/>
+<wire x1="144.78" y1="45.72" x2="144.78" y2="53.34" width="0.1524" layer="91"/>
 </segment>
 </net>
@@
 </segment>
 </net>
+<net name="N$5" class="0">
+<segment>
+<pinref part="IC1" gate="PORTD/OSC" pin="PD1/OSC=&gt;"/>
+<pinref part="R3" gate="G$1" pin="1"/>
+<wire x1="121.92" y1="55.88" x2="129.54" y2="55.88" width="0.1524" layer="91"/>
+<wire x1="129.54" y1="55.88" x2="129.54" y2="45.72" width="0.1524" layer="91"/>
+</segment>
+</net>
+<net name="N$3" class="0">
+<segment>
+<pinref part="IC1" gate="RESET" pin="BOOT0"/>
+<pinref part="R4" gate="G$1" pin="1"/>
+<wire x1="121.92" y1="144.78" x2="121.92" y2="137.16" width="0.1524" layer="91"/>
+</segment>
+</net>
+<net name="N$6" class="0">
+<segment>
+<pinref part="R4" gate="G$1" pin="2"/>
+<pinref part="S1" gate="1" pin="P"/>
+<wire x1="132.08" y1="137.16" x2="134.62" y2="137.16" width="0.1524" layer="91"/>
+</segment>
+</net>
